Commit message: update

File: fts300s_description/urdf/robotiq_fts300s.urdf.xacro (robot description, xacro)
@@ -17,5 +17,5 @@
                 <origin xyz="0 0 0.035851" rpy="${-pi} 0 0" />
                 <geometry>
-                    <mesh filename="package://robotiq_ft_sensor/meshes/visual/fts300s.stl" scale="0.001 0.001 0.001"/>
+                    <mesh filename="package://fts300s_description/meshes/visual/fts300s.stl" scale="0.001 0.001 0.001"/>
                 </geometry>
                 <material name="black"/>
@@ -24,5 +24,5 @@
                 <origin xyz="0 0 0.035851" rpy="${-pi} 0 0" />
                 <geometry>
-                    <mesh filename="package://robotiq_ft_sensor/meshes/collision/fts300s.stl" scale="0.001 0.001 0.001"/>
+                    <mesh filename="package://fts300s_description/meshes/collision/fts300s.stl" scale="0.001 0.001 0.001"/>
                 </geometry>
             </collision>

Commit message: Modifications

File: fts300s_description/urdf/robotiq_fts300s.urdf.xacro (robot description, xacro)
@@ -28,11 +28,4 @@
             </collision>
         </link>
-        <!-- virtual measurement frame -->
-        <joint name="${prefix}measurment_joint" type="fixed" >
-            <origin xyz="0 0 0.01625" rpy="0 0 0" />
-            <parent link="${prefix}fts_robotside" />
-            <child link="${prefix}robotiq_force_torque_frame_id" />
-        </joint>
-        <link name="${prefix}robotiq_force_torque_frame_id"/>
         <!-- toolside frame -->
         <joint name="${prefix}toolside_joint" type="fixed" >
