Commit message: Modification

File: ft300s_description/urdf/robotiq_fts300s.urdf.xacro (robot description, xacro)
@@ -17,5 +17,5 @@
                 <origin xyz="0 0 0.035851" rpy="${-pi} 0 0" />
                 <geometry>
-                    <mesh filename="package://fts300s_description/meshes/visual/fts300s.stl" scale="0.001 0.001 0.001"/>
+                    <mesh filename="package://ft300s_description/meshes/visual/fts300s.stl" scale="0.001 0.001 0.001"/>
                 </geometry>
                 <material name="black"/>
@@ -24,5 +24,5 @@
                 <origin xyz="0 0 0.035851" rpy="${-pi} 0 0" />
                 <geometry>
-                    <mesh filename="package://fts300s_description/meshes/collision/fts300s.stl" scale="0.001 0.001 0.001"/>
+                    <mesh filename="package://ft300s_description/meshes/collision/fts300s.stl" scale="0.001 0.001 0.001"/>
                 </geometry>
             </collision>
@@ -31,8 +31,8 @@
         <joint name="${prefix}toolside_joint" type="fixed" >
             <origin xyz="0 0 0.03851" rpy="0 0 0" />
-            <parent link="${prefix}fts_robotside" />
-            <child link="${prefix}fts_toolside" />
+            <parent link="${prefix}ft_robotside" />
+            <child link="${prefix}ft_toolside" />
         </joint>
-        <link name="${prefix}fts_toolside"/>
+        <link name="${prefix}ft_toolside"/>
     </xacro:macro>
 </robot>
